File: Isolated dual rail PS controlled submodule.kicad_sch (KiCad schematic)
At the start: 7 parts, among them U10 TPS1H100BQPWPRQ1, U11 TPS1H100BQPWPRQ1, U12 TPS1H100BQPWPRQ1, U2 INA4235AIYBJR, U7 TPL0102-100PWR, U8 TPL0102-100PWR, U9 TPS1H100BQPWPRQ1

Commit message: HW-61 chore: FT4233 Wire'd up
Parts:
- removed U10, U11, U12, U9: TPS1H100BQPWPRQ1, semiconductor:HTSSOP-14-1EP_P0.65_4.4x5x1.2, symbol integrated-circuit:TPS1H100BQPWPRQ1
- removed U8: TPL0102-100PWR, semiconductor:TSSOP-14_P0.65_4.4x5x1.2, symbol integrated-circuit:TPL0102-100PWR
- added C100, C83, C84, C96, C97, C99: 1uF-0402_01, passive:Capacitor_0402, symbol capacitor:1uF-0402_01
- added C81, C82, C87, C89: 10uF-0603_01, passive:Capacitor_0603, symbol capacitor:10uF-0603_01
- added C85: 3.3uF-0603_01, passive:Capacitor_0603, symbol capacitor:3.3uF-0603_01
- added C86, C88: 22uF-0603_01, passive:Capacitor_0603, symbol capacitor:22uF-0603_01
- added C90, C91, C92: 220nF-0402_02, passive:Capacitor_0402, symbol staging:220nF-0402_02
- added C93, C94, C95: 22nF-0805_01, passive:Capacitor_0805, symbol capacitor:22nF-0805_01
- added C98: 100nF-0402_01, passive:Capacitor_0402, symbol capacitor:100nF-0402_01
- added R56: 10k-0402_02, passive:Resistor_0402, symbol resistor:10k-0402_02
- added R57, R58, R59: 1k-0402_01, passive:Resistor_0402, symbol resistor:1k-0402_01
- added R60, R61, R62, R63, R64, R65, R66, R67: 0R-0402_01, passive:Resistor_0402, symbol resistor:0R-0402_01
- added U31: TPS7A3301RGWR, semiconductor:VQFN-20-1EP_P0.65_5x5x1, symbol staging:TPS7A3301RGWR
- added U32: TPS7A4701QRGWTQ1, semiconductor:VQFN-20-1EP_P0.65_5x5x1, symbol staging:TPS7A4701QRGWTQ1
- added U34, U35, U36: TPS1HTC30AQPWPRQ1, semiconductor:HTSSOP-14-1EP_P0.65_4.4x5x1.2, symbol staging:TPS1HTC30AQPWPRQ1
- renumbered U7 to U33, U2 to U37
Connections:
- net +15V_ISO: now also C82.1, U32.13 (EN), U32.15 (IN), U32.16 (IN)
- net +PWR_SWITCH_ISO_1X_EN: now also U35.2 (EN)
- net +PWR_SWITCH_ISO_2X_EN: now also U34.2 (EN)
- net -15V_ISO: now also C81.1, U31.13 (EN), U31.15 (IN), U31.16 (IN)
- net -PWR_SWITCH_ISO_2X_EN: now also U36.2 (EN)
- net Current shunt/INPUT_CURRENT: now also C93.1, U34.10 (VOUT), U34.8 (VOUT), U34.9 (VOUT)
- net Current shunt1/INPUT_CURRENT: now also C94.1, U35.10 (VOUT), U35.8 (VOUT), U35.9 (VOUT)
- net +15V_LDO: now reaches U33.1 (HA)
- net +15V_LDO: now also C87.1, C89.1, C90.1, C91.1, U32.1 (OUT), U32.20 (OUT), U34.12 (VS), U34.13 (VS), U34.14 (VS), U35.12 (VS), U35.13 (VS), U35.14 (VS)
- net GND_ISO_15V: now reaches U33.11 (GND)
- net GND_ISO_15V: now also U33.8 (VSS), U37.B4 (GND), C81.2, C82.2, C83.2, C84.2, C85.2, C86.2, C87.2, C88.2, C89.2, C90.2, C91.2, C92.2, C93.2, C94.2, C95.2, R56.1, R57.1, R58.1, R59.1, U31.7 (GND), U32.7 (GND), U34.1 (GND), U34.15 (Thermal_Pad), U35.1 (GND), U35.15 (Thermal_Pad), U36.1 (GND), U36.15 (Thermal_Pad)
- net VDD_ISO_3: now reaches U33.14 (VDD)
- net VDD_ISO_3: now also U37.A4 (VS), U37.B3 (EN), C98.1
- net +15V_LDO_V_SENSE: now reaches U33.2 (LA)
- net +15V_LDO_V_SENSE: now also U33.3 (WA)
- net -15V_LDO: now reaches U33.4 (HB)
- net -15V_LDO: now also C85.1, C86.1, C88.1, C92.1, U31.1 (OUT), U31.20 (OUT), U36.12 (VS), U36.13 (VS), U36.14 (VS)
- net -15V_LDO_V_SENSE: now reaches U33.5 (LB)
- net -15V_LDO_V_SENSE: now also U33.6 (WB)
- net at U37.A1 (IN+2): now also R62.2
- net at U37.A2 (IN-1): now also R61.2
- net at U37.A3 (IN+1): now also R60.2
- net at U37.B1 (IN-2): now also R63.2
- net at U37.C1 (IN-3): now also R65.1
- net at U37.D1 (IN+3): now also R64.1
- net at U37.D2 (IN-4): now also R67.1
- net at U37.D3 (IN+4): now also R66.1
- net SCK_ISO renamed SCL_ISO
- new net: R59.2, U36.6 (SNS)
- new net: C84.1, U32.14 (NR)
- new net: C95.1, U36.10 (VOUT), U36.8 (VOUT), U36.9 (VOUT)
- new net: R57.2, U34.6 (SNS)
- new net: R58.2, U35.6 (SNS)
- new net: C100.1, R66.2
- new net: C99.1, R64.2
- new net: C100.2, R67.2
- new net: C83.1, U31.14 (NR)
- new net: C99.2, R65.2
- new net +INA_DRAIL_1: C96.1, R60.1
- new net +INA_DRAIL_2: C97.1, R62.1
- new net -INA_DRAIL_1: C96.2, R61.1
- new net -INA_DRAIL_2: C97.2, R63.1
- new net 15V_LDO_V_SENSE: R56.2, U32.3 (SENSE/FB)
- new net GND: C98.2
- no-connect marks 0 -> 21
Other:
- moved on the sheet: U33, U37A

Commit message: Details to finish
Parts:
- removed C92: 220nF-0402_02, passive:Capacitor_0402, symbol staging:220nF-0402_02
- removed C95: 22nF-0805_01, passive:Capacitor_0805, symbol capacitor:22nF-0805_01
- removed R59: 1k-0402_01, passive:Resistor_0402, symbol resistor:1k-0402_01
- removed U36: TPS1HTC30AQPWPRQ1, semiconductor:HTSSOP-14-1EP_P0.65_4.4x5x1.2, symbol staging:TPS1HTC30AQPWPRQ1
- added C214, C92: 1uF-0402_01, passive:Capacitor_0402, symbol capacitor:1uF-0402_01
- added C217, C219: 100nF-0402_01, passive:Capacitor_0402, symbol capacitor:100nF-0402_01
- added Q13, Q17: MMBT2907A, semiconductor:SOT23-3_P0.95_2.92x1.3x1.12, symbol semiconductor:MMBT2907A
- added Q16, Q20: SI7110DN-T1-GE3, staging:PowerPAK-8_P0.66_3.3x3.3x1.04, symbol staging:SIA440DJ-T1-GE3
- added Q22, Q25, Q27: RK7002BM, semiconductor:SOT-23-3-INV_P0.95_2.92x1.3x1.12, symbol semiconductor:RK7002BM
- added R170, R59: 100R-0402_01, passive:Resistor_0402, symbol resistor:100R-0402_01
- added R171, R197, R199, R227, R229, R233, R71: 1k-0402_01, passive:Resistor_0402, symbol resistor:1k-0402_01
- added R172, R181: 10k-0402_02, passive:Resistor_0402, symbol resistor:10k-0402_02
- added R173, R182, R219, R221, R223: 1M-0402_01, passive:Resistor_0402, symbol resistor:1M-0402_01
- added R215, R217: 499k-0402_01, passive:Resistor_0402, symbol resistor:499k-0402_01
- added R225: 215k-0402_01, passive:Resistor_0402, symbol resistor:215k-0402_01
- added R231: 715k-0402_01, passive:Resistor_0402, symbol resistor:715k-0402_01
Connections:
- net -15V_LDO: now also Q16.4 (S), Q16.7 (S), Q20.4 (S), Q20.7 (S), R172.2, R181.2, R225.2
- net Current shunt2/INPUT_CURRENT: now also C217.1, Q16.1 (D), Q16.2 (D), Q16.5 (D), Q16.6 (D), R173.2
- net Current shunt3/INPUT_CURRENT: now also C219.1, Q20.1 (D), Q20.2 (D), Q20.5 (D), Q20.6 (D), R182.2
- net GND_ISO_15V: now also C214.1, C217.2, C219.2, C92.2, R173.1, R182.1, R215.1, R217.1, R231.1
- net SCL_ISO: now also U37.C4 (SCL)
- net SDA_ISO: now also U37.D4 (SDA)
- net VDD_ISO_3: now also Q13.2 (E), Q17.2 (E), R197.2, R199.2
- net +INA_CTRL_RAIL_4: now reaches C100.1, R66.2
- net +INA_CTRL_RAIL_3: now reaches C99.1, R64.2
- net -INA_CTRL_RAIL_4: now reaches C100.2, R67.2
- net FB_SELECT: now reaches U31.3 (SENSE/FB)
- net FB_SELECT: now also Q22.3 (D), Q25.3 (D), Q27.3 (D), R225.1
- net INA_A0: now reaches U37.C2 (A0)
- net INA_A1: now reaches U37.C3 (A1)
- net -INA_CTRL_RAIL_3: now reaches C99.2, R65.2
- net +INA_DRAIL_1 renamed +INA_CTRL_RAIL_1
- net +INA_DRAIL_2 renamed +INA_CTRL_RAIL_2
- net +PWR_SWITCH_ISO_1X_EN renamed +PWR_SWITCH_ISO_CTRL_X2_EN
- net +PWR_SWITCH_ISO_2X_EN renamed +PWR_SWITCH_ISO_CTRL_X1_EN
- net -INA_DRAIL_1 renamed -INA_CTRL_RAIL_1
- net -INA_DRAIL_2 renamed -INA_CTRL_RAIL_2
- new net: R215.2, R219.1
- new net: R221.2, R223.1
- new net: Q22.1 (S), R223.2, R227.1
- new net: C214.2, Q13.1 (B), R170.2
- new net: Q25.1 (S), R219.2, R229.1
- new net: Q25.2 (G), R229.2
- new net: Q22.2 (G), R227.2
- new net: R217.2, R221.1
- new net: C92.1, Q17.1 (B), R59.2
- new net: Q17.3 (C), R71.1
- new net: Q20.3 (G), R181.1, R71.2
- new net: Q13.3 (C), R171.1
- new net: Q27.1 (S), R231.2, R233.1
- new net: Q27.2 (G), R233.2
- new net: Q16.3 (G), R171.2, R172.1
- new net -PWR_SWITCH_ISO_CTRL_1X_EN: R170.1, R197.1
- new net -PWR_SWITCH_ISO_CTRL_2X_EN: R199.1, R59.1
- no-connect marks 21 -> 17
Other:
- moved on the sheet: C100, C81, C82, C83, C84, C85, C86, C87, C88, C89, C90, C91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
