File: Isolated dual rail PS controlled submodule.kicad_sch (KiCad schematic)
At the start: 66 parts, among them Q13 MMBT2907A, Q16 SI7110DN-T1-GE3, Q17 MMBT2907A, Q20 SI7110DN-T1-GE3, Q22 RK7002BM, Q25 RK7002BM, Q27 RK7002BM, U31 TPS7A3301RGWR, U32 TPS7A4701QRGWTQ1, U33 TPL0102-100PWR, U34 TPS1HTC30AQPWPRQ1, U35 TPS1HTC30AQPWPRQ1, U37 INA4235AIYBJR

Commit message: HW-61/chore: Added simulation for switch ocntrol, organized the overall schematic, fixed the ERC errors. Still pending for the current sense components and negative side LDO control
Parts:
- removed C214, C92: 1uF-0402_01, passive:Capacitor_0402, symbol capacitor:1uF-0402_01
- removed Q22, Q25, Q27: RK7002BM, semiconductor:SOT-23-3-INV_P0.95_2.92x1.3x1.12, symbol semiconductor:RK7002BM
- removed R215, R217: 499k-0402_01, passive:Resistor_0402, symbol resistor:499k-0402_01
- removed R219, R221, R223: 1M-0402_01, passive:Resistor_0402, symbol resistor:1M-0402_01
- removed R227, R229, R233: 1k-0402_01, passive:Resistor_0402, symbol resistor:1k-0402_01
- removed R231: 715k-0402_01, passive:Resistor_0402, symbol resistor:715k-0402_01
- added C111, C92: 100nF-0402_01, passive:Capacitor_0402, symbol capacitor:100nF-0402_01
- added R241, R243: 1k-0402_01, passive:Resistor_0402, symbol resistor:1k-0402_01
Connections:
- net +PWR_SWITCH_ISO_CTRL_X1_EN: now also R241.2
- net +PWR_SWITCH_ISO_CTRL_X2_EN: now also R243.2
- net GND_ISO_15V: now also C111.2, C92.2, R241.1, R243.1
- net at Q13.1 (B), R170.2: now also C111.1
- net DigiPot_A1: now reaches U33.12 (A1)
- net DigiPot_A0: now reaches U33.13 (A0)
- net DigiPot_A2: now reaches U33.7 (A2)
- net at Q17.1 (B), R59.2: now also C92.1
- net -PWR_SWITCH_ISO_CTRL_1X_EN renamed ~{-PWR_SWITCH_ISO_CTRL_1X_EN}
- net -PWR_SWITCH_ISO_CTRL_2X_EN renamed ~{-PWR_SWITCH_ISO_CTRL_2X_EN}
Other:
- moved on the sheet: C217, C219, R197, U33
