File: Buck stage.kicad_sch (KiCad schematic)
At the start: 1 part, among them U16 PCA9535PWR

Commit message: HW-61 chore: FT4233 Wire'd up
Parts:
- added U10, U11: TPL0102-100PWR, semiconductor:TSSOP-14_P0.65_4.4x5x1.2, symbol integrated-circuit:TPL0102-100PWR
- added U13: PCA9535PWR, semiconductor:TSSOP-24_P0.65_7.8x4.4x1.2, symbol integrated-circuit:PCA9535PWR
- renumbered U16 to U12
Connections:
- net Buck submodule/PWR_SWITCH_EN_1: now also U12.4 (P00_B)
- net Buck submodule/PWR_SWITCH_EN_2: now also U12.5 (P01_B)
- net Buck submodule/PWR_SWITCH_EN_3: now also U12.6 (P02_B)
- net Buck submodule/PWR_SWITCH_EN_4: now also U12.7 (P03_B)
- net Buck submodule1/PWR_SWITCH_EN_1: now also U12.8 (P04_B)
- net Buck submodule1/PWR_SWITCH_EN_2: now also U12.9 (P05_B)
- net Buck submodule1/PWR_SWITCH_EN_3: now also U12.10 (P06_B)
- net Buck submodule1/PWR_SWITCH_EN_4: now also U12.11 (P07_B)
- net Buck submodule2/PWR_SWITCH_EN_1: now also U12.13 (P10_B)
- net Buck submodule2/PWR_SWITCH_EN_2: now also U12.14 (P11_B)
- net Buck submodule2/PWR_SWITCH_EN_3: now also U12.15 (P12_B)
- net Buck submodule2/PWR_SWITCH_EN_4: now also U12.16 (P13_B)
- net Buck submodule3/PWR_SWITCH_EN_1: now also U12.17 (P14_B)
- net Buck submodule3/PWR_SWITCH_EN_2: now also U12.18 (P15_B)
- net Buck submodule3/PWR_SWITCH_EN_3: now also U12.19 (P16_B)
- net Buck submodule3/PWR_SWITCH_EN_4: now also U12.20 (P17_B)
- net GND: now reaches U12.12 (GND)
- net GND: now also U12.2 (A1), U12.21 (A0), U12.3 (A2), U10.11 (GND), U10.12 (A1), U10.13 (A0), U10.7 (A2), U10.8 (VSS), U11.11 (GND), U11.12 (A1), U11.7 (A2), U13.12 (GND), U13.2 (A1), U13.21 (A0)
- net SCL: now reaches U12.22 (SCL)
- net SCL: now also U10.10 (SCL), U11.10 (SCL), U13.22 (SCL)
- net SDA: now reaches U12.23 (SDA)
- net SDA: now also U10.9 (SDA), U11.9 (SDA), U13.23 (SDA)
- net +5V: now reaches U12.24 (VDD)
- net +5V: now also U10.14 (VDD), U11.13 (A0), U11.14 (VDD), U13.24 (VDD), U13.3 (A2)
- new net BUCK_SUBMODULE_1_IN: U10.1 (HA)
- new net BUCK_SUBMODULE_1_OUT: U10.2 (LA), U10.3 (WA)
- new net BUCK_SUBMODULE_2_IN: U10.4 (HB)
- new net BUCK_SUBMODULE_2_OUT: U10.5 (LB), U10.6 (WB)
- new net BUCK_SUBMODULE_3_IN: U11.1 (HA)
- new net BUCK_SUBMODULE_3_OUT: U11.2 (LA), U11.3 (WA)
- new net BUCK_SUBMODULE_4_IN: U11.4 (HB)
- new net BUCK_SUBMODULE_4_OUT: U11.5 (LB), U11.6 (WB)
- new net Buck submodule/SCALE_BUCK_1: U13.4 (P00_B)
- new net Buck submodule/SCALE_BUCK_2: U13.5 (P01_B)
- new net Buck submodule/SCALE_BUCK_3: U13.6 (P02_B)
- new net Buck submodule/SCALE_BUCK_4: U13.7 (P03_B)
- new net Buck submodule1/SCALE_BUCK_1: U13.8 (P04_B)
- new net Buck submodule1/SCALE_BUCK_2: U13.9 (P05_B)
- new net Buck submodule1/SCALE_BUCK_3: U13.10 (P06_B)
- new net Buck submodule1/SCALE_BUCK_4: U13.11 (P07_B)
- new net Buck submodule2/SCALE_BUCK_1: U13.13 (P10_B)
- new net Buck submodule2/SCALE_BUCK_2: U13.14 (P11_B)
- new net Buck submodule2/SCALE_BUCK_3: U13.15 (P12_B)
- new net Buck submodule2/SCALE_BUCK_4: U13.16 (P13_B)
- new net Buck submodule3/SCALE_BUCK_1: U13.17 (P14_B)
- new net Buck submodule3/SCALE_BUCK_2: U13.18 (P15_B)
- new net Buck submodule3/SCALE_BUCK_3: U13.19 (P16_B)
- new net Buck submodule3/SCALE_BUCK_4: U13.20 (P17_B)
- no-connect marks 0 -> 2
Other:
- sheet Buck submodule ports: added FB_RESISTOR_IN, FB_RESISTOR_OUT, INA_A0, INA_A1, SCALE_BUCK_1, SCALE_BUCK_2, SCALE_BUCK_3, SCALE_BUCK_4; removed none
- sheet Buck submodule1 ports: added FB_RESISTOR_IN, FB_RESISTOR_OUT, INA_A0, INA_A1, SCALE_BUCK_1, SCALE_BUCK_2, SCALE_BUCK_3, SCALE_BUCK_4; removed none
- sheet Buck submodule2 ports: added FB_RESISTOR_IN, FB_RESISTOR_OUT, INA_A0, INA_A1, SCALE_BUCK_1, SCALE_BUCK_2, SCALE_BUCK_3, SCALE_BUCK_4; removed none
- sheet Buck submodule3 ports: added FB_RESISTOR_IN, FB_RESISTOR_OUT, INA_A0, INA_A1, SCALE_BUCK_1, SCALE_BUCK_2, SCALE_BUCK_3, SCALE_BUCK_4; removed none
- note added: "I2C ID: 0x20"
- note added: "I2C ID: 0x21"
- note added: "I2C ID: 0x50"
- note added: "I2C ID: 0x51"
- note added: "INA I2C ID: 0x40"
- note added: "INA I2C ID: 0x41"
- note added: "INA I2C ID: 0x42"
- note added: "INA I2C ID: 0x43"
- moved on the sheet: U12

Commit message: Details to finish
Connections:
- net BUCK_SUBMODULE_2_OUT is gone; now on net BUCK_SUBMODULE_2_IN: U10.5 (LB), U10.6 (WB)
- net Buck submodule1/PWR_SWITCH_EN_4 is gone; now on net BUCK_SUBMODULE_2_IN: U12.11 (P07_B)
Other:
- note added: "4x Bucks output voltage control (DigiPot)"
- note added: "4x Bucks submodules"
- note added: "I/O Mux Channel Enable control"
- moved on the sheet: U10, U11, U12, U13

Commit message: HW-61/chore: Added simulation for switch ocntrol, organized the overall schematic, fixed the ERC errors. Still pending for the current sense components and negative side LDO control
Connections:
- net +5V: now also U13.21 (A0); no longer U13.3 (A2)
- net GND: now also U11.8 (VSS), U13.3 (A2); no longer U13.21 (A0)
- net SCL renamed SCL_A
- net SDA renamed SDA_A
Other:
- note removed: "I/O Mux Channel Enable control"
- moved on the sheet: U12
