File: Isolated dual rail fixed PS stage.kicad_sch (KiCad schematic)
At the start: 8 parts, among them U18 INA2227AIYBJR, U19 INA2227AIYBJR, U20 INA2227AIYBJR, U21 ADM3260ARSZ-RL7, U22 ADM3260ARSZ-RL7

Commit message: HW-61 chore: FT4233 Wire'd up
Parts:
- removed U18, U19, U20: INA2227AIYBJR, digikey:U_BGA_YBJ0016-C01_TEX-M, symbol digikey:INA2227AIYBJR
- removed U21, U22: ADM3260ARSZ-RL7, digikey:SSOP-20_RS-20_ADI-M, symbol integrated-circuit:ADM3260ARSZ-RL7
- added C39, C41, C43, C51, C52, C53: 10uF-0402_01, passive:Capacitor_0402, symbol capacitor:10uF-0402_01
- added C40, C42, C44, C45, C46, C47, C48, C49, C50, C66, C67, C68, C69, C70, C71: 100nF-0402_01, passive:Capacitor_0402, symbol capacitor:100nF-0402_01
- added C54, C55, C56: 150uF-7343-43, tantalumCaps:CP_EIA-7343-43_Kemet-X, symbol staging:150uF-7343-43
- added C57, C58, C59: 10uF-0603_01, passive:Capacitor_0603, symbol capacitor:10uF-0603_01
- added C60, C61, C62, C63, C64, C65: 10uF-1210_01, passive:Capacitor_Polarized_EIA_3528-21, symbol staging:10uF-1210_01
- added C72, C73, C74: 220nF-0402_02, passive:Capacitor_0402, symbol staging:220nF-0402_02
- added C75, C76, C77: 22nF-0805_01, passive:Capacitor_0805, symbol capacitor:22nF-0805_01
- added C78, C79, C80: 10nF-0402_01, passive:Capacitor_0402, symbol capacitor:10nF-0402_01
- added L1, L2, L3: 10uH-3.2x2.5x1.2_01, passive:TFM322512ALMA, symbol inductor:10uH-3.2x2.5x1.2_01
- added R35, R37, R39: 30.9k-0402_01, passive:Resistor_0402, symbol staging:30.9k-0402_01
- added R36, R38, R40: 10k-0402_02, passive:Resistor_0402, symbol resistor:10k-0402_02
- added R41, R42, R43, R44, R45, R46: 4.7k-0402_01, passive:Resistor_0402, symbol resistor:4.7k-0402_01
- added R47, R48, R49: 0R-0402_01, passive:Resistor_0402, symbol resistor:0R-0402_01
- added R50, R51, R52: 100k-0402_01, passive:Resistor_0402, symbol resistor:100k-0402_01
- added R53, R54, R55: 1k-0402_01, passive:Resistor_0402, symbol resistor:1k-0402_01
- added U20, U21, U22: ADM3260ARSZ-RL7, digikey:SSOP-20_P0.65_7.2x5.3mm, symbol staging:ADM3260ARSZ-RL7
- added U23, U24, U25: TPS1HTC30AQPWPRQ1, semiconductor:HTSSOP-14-1EP_P0.65_4.4x5x1.2, symbol staging:TPS1HTC30AQPWPRQ1
- added U26, U27: TLP291-4GB-TP_E, digikey:SO-16_TOS_P1.27_10.45x4.6mm, symbol staging:TLP291-4GB-TP_E
- added U28, U29, U30: INA2227AIYBJR, review:DSBGA-16_P0.4_1.508X1.508mm, symbol staging:INA2227AIYBJR
Connections:
- net 12V_EN: now also PS2.3 (CTRL), R51.2
- net 15V_EN: now also PS3.3 (CTRL), R52.2
- net 5V_EN: now also PS1.3 (CTRL), R50.2
- net GND: now also PS1.2 (-Vin), PS2.2 (-Vin), PS3.2 (-Vin), C39.2, C40.2, C41.2, C42.2, C43.2, C44.2, C45.2, C46.2, C47.2, C54.2, C55.2, C56.2, C57.2, C58.2, C59.2, R50.1, R51.1, R52.1, U20.1 (GNDP), U20.10 (GNDP), U20.5 (GNDP), U20.7 (GNDP), U20.8 (PDIS), U21.1 (GNDP), U21.10 (GNDP), U21.5 (GNDP), U21.7 (GNDP), U21.8 (PDIS), U22.1 (GNDP), U22.10 (GNDP), U22.5 (GNDP), U22.7 (GNDP), U22.8 (PDIS)
- net at PS1.1 (+Vin): now also C57.1, L1.2, R47.2
- net -5V_ISO: now reaches PS1.4 (-Vout)
- net -5V_ISO: now also C63.2, C69.2
- net GND_ISO_5V: now reaches PS1.5 (COM)
- net GND_ISO_5V: now also C48.2, C51.2, C62.2, C63.1, C68.2, C69.1, C72.2, C75.2, R36.1, R53.1, U20.11 (GNDISO), U20.14 (GNDISO), U20.16 (GNDISO), U20.20 (GNDISO), U23.1 (GND), U23.15 (Thermal_Pad), U28.B4 (GND)
- net +5V_ISO: now reaches PS1.6 (+Vou)
- net +5V_ISO: now also C62.1, C68.1, C72.1, U23.12 (VS), U23.13 (VS), U23.14 (VS)
- net at PS2.1 (+Vin): now also C58.1, L2.2, R48.2
- net -12V_ISO: now reaches PS2.4 (-Vout)
- net -12V_ISO: now also C65.2, C71.2
- net GND_ISO_12V: now reaches PS2.5 (COM)
- net GND_ISO_12V: now also C49.2, C52.2, C64.2, C65.1, C70.2, C71.1, C73.2, C76.2, R38.1, R54.1, U21.11 (GNDISO), U21.14 (GNDISO), U21.16 (GNDISO), U21.20 (GNDISO), U24.1 (GND), U24.15 (Thermal_Pad), U29.B4 (GND)
- net +12V_ISO: now reaches PS2.6 (+Vou)
- net +12V_ISO: now also C64.1, C70.1, C73.1, U24.12 (VS), U24.13 (VS), U24.14 (VS)
- net at PS3.1 (+Vin): now also C59.1, L3.2, R49.2
- net -15V_ISO: now reaches PS3.4 (-Vout)
- net -15V_ISO: now also C61.2, C67.2
- net GND_ISO_15V: now reaches PS3.5 (COM)
- net GND_ISO_15V: now also C50.2, C53.2, C60.2, C61.1, C66.2, C67.1, C74.2, C77.2, R40.1, R55.1, U22.11 (GNDISO), U22.14 (GNDISO), U22.16 (GNDISO), U22.20 (GNDISO), U25.1 (GND), U25.15 (Thermal_Pad), U30.B4 (GND)
- net +15V_ISO: now reaches PS3.6 (+Vou)
- net +15V_ISO: now also C60.1, C66.1, C74.1, U25.12 (VS), U25.13 (VS), U25.14 (VS)
- new net: R35.1, R36.2, U20.13 (VSEL)
- new net: C76.1, U24.10 (VOUT), U24.8 (VOUT), U24.9 (VOUT)
- new net: R54.2, U24.6 (SNS)
- new net: C77.1, U25.10 (VOUT), U25.8 (VOUT), U25.9 (VOUT)
- new net: R55.2, U25.6 (SNS)
- new net: C75.1, U23.10 (VOUT), U23.8 (VOUT), U23.9 (VOUT)
- new net: R39.1, R40.2, U22.13 (VSEL)
- new net: R53.2, U23.6 (SNS)
- new net: R37.1, R38.2, U21.13 (VSEL)
- new net +24V: C54.1, C55.1, C56.1, L1.1, L2.1, L3.1, R47.1, R48.1, R49.1
- new net +5V: C39.1, C40.1, C41.1, C42.1, C43.1, C44.1, C45.1, C46.1, C47.1, U20.4 (VDDP), U20.9 (VIN), U21.4 (VDDP), U21.9 (VIN), U22.4 (VDDP), U22.9 (VIN)
- new net 12V_SCL_ISO: R42.1, U21.19 (SCL1), U29.C4 (SCL), U30.C4 (SCL)
- new net 12V_SDA_ISO: R45.1, U21.18 (SDA1), U29.D4 (SDA), U30.D4 (SDA)
- new net 15V_SCL_ISO: R43.1, U22.19 (SCL1)
- new net 15V_SDA_ISO: R46.1, U22.18 (SDA1)
- new net 5V_SCL_ISO: R41.1, U20.19 (SCL1), U28.C4 (SCL)
- new net 5V_SDA_ISO: R44.1, U20.18 (SDA1), U28.D4 (SDA)
- new net SCL: U20.2 (SCL2), U21.2 (SCL2), U22.2 (SCL2)
- new net SDA: U20.3 (SDA2), U21.3 (SDA2), U22.3 (SDA2)
- new net VDD_ISO_1: C48.1, C51.1, C78.1, C78.2, R35.2, R41.2, R44.2, U20.12 (VISO), U20.12 (VISO), U20.17 (VDDISO), U28.A4 (VS), U28.B3 (EN)
- new net VDD_ISO_2: C49.1, C52.1, C79.1, C79.2, R37.2, R42.2, R45.2, U21.12 (VISO), U21.12 (VISO), U21.17 (VDDISO), U29.A4 (VS), U29.B3 (EN)
- new net VDD_ISO_3: C50.1, C53.1, C80.1, C80.2, R39.2, R43.2, R46.2, U22.12 (VISO), U22.12 (VISO), U22.17 (VDDISO), U30.A4 (VS), U30.B3 (EN)
- no-connect marks 0 -> 15
Other:
- added sheet Isolated dual rail PS controlled submodule (Isolated dual rail PS controlled submodule.kicad_sch)
- added sheet Isolated dual rail PS controlled submodule1 (Isolated dual rail PS controlled submodule.kicad_sch)
- note added: "Needs to set the I2C ID"
- moved on the sheet: PS1, PS2, PS3

Commit message: Details to finish
Parts:
- removed C78, C79, C80: 10nF-0402_01, passive:Capacitor_0402, symbol capacitor:10nF-0402_01
- added C112, C115, C216, C78, C79, C80: 100nF-0402_01, passive:Capacitor_0402, symbol capacitor:100nF-0402_01
- added C211, C212, C213: 1uF-0402_01, passive:Capacitor_0402, symbol capacitor:1uF-0402_01
- added Q10, Q12: SI7110DN-T1-GE3, staging:PowerPAK-8_P0.66_3.3x3.3x1.04, symbol staging:SIA440DJ-T1-GE3
- added Q11, Q23, Q9: MMBT2907A, semiconductor:SOT23-3_P0.95_2.92x1.3x1.12, symbol semiconductor:MMBT2907A
- added Q14: SI4866DY-T1-GE3, staging:SO-8_P_1.27_3.9x4.9x1.55, symbol staging:SI4866DY-T1-GE3
- added R161, R164, R167, R187, R188, R195, R196, R201, R202, R205, R206, R207, R208, R211, R212: 100R-0402_01, passive:Resistor_0402, symbol resistor:100R-0402_01
- added R162, R166, R169: 10k-0402_02, passive:Resistor_0402, symbol resistor:10k-0402_02
- added R163, R165, R168, R189, R190, R191, R192, R193, R194, R203, R204, R209, R210, R213, R214: 1k-0402_01, passive:Resistor_0402, symbol resistor:1k-0402_01
- added R176, R177, R178: 1M-0402_01, passive:Resistor_0402, symbol resistor:1M-0402_01
- added U36: TLP291-4GB-TP_E, digikey:SO-16_TOS_P1.27_10.45x4.6mm, symbol staging:TLP291-4GB-TP_E
- added U43, U67: PCA9535PWR, semiconductor:TSSOP-24_P0.65_7.8x4.4x1.2, symbol integrated-circuit:PCA9535PWR
Connections:
- net +5V: now also R203.2, R204.2, R209.2, R210.2, R213.2, R214.2, U43.24 (VDD), U67.24 (VDD)
- net -12V_ISO: now also Q10.4 (S), Q10.7 (S), R162.2
- net -15V_ISO: now also Q12.4 (S), Q12.7 (S), R166.2
- net -5V_ISO: now also Q14.1 (S), Q14.2 (S), Q14.3 (S), R169.2
- net 12V_SDA_ISO: now also U30.D3 (A0)
- net Current shunt1/INPUT_CURRENT: now also C76.1, U24.10 (VOUT), U24.8 (VOUT), U24.9 (VOUT)
- net Current shunt4/INPUT_CURRENT: now also C77.1, U25.10 (VOUT), U25.8 (VOUT), U25.9 (VOUT)
- net Current shunt5/INPUT_CURRENT: now also C216.1, Q14.5 (D), Q14.6 (D), Q14.7 (D), Q14.8 (D), R176.2
- net GND: now also U26.6, U26.8, U27.6, U27.8, U36.6, U36.8, U43.12 (GND), U67.12 (GND)
- net GND_ISO_12V: now also U27.2, U27.4, U27.9, C115.2, C211.2, C79.2, R177.1, R193.1
- net GND_ISO_15V: now also C112.2, C212.2, C80.2, R178.1, R194.1, U36.2, U36.4, U36.9
- net GND_ISO_5V: now also U26.2, U26.4, U26.9, U28.D3 (A0), C213.2, C216.2, C78.2, R176.1, R189.1
- net SCL: now also U43.22 (SCL), U67.22 (SCL)
- net SDA: now also U43.23 (SDA), U67.23 (SDA)
- net VDD_ISO_1: now also U26.12, U28.A2 (VBUS1), U28.C3 (A1), U28.D2 (VBUS2), C78.1, Q23.2 (E), R190.2
- net VDD_ISO_2: now also U27.12, U29.A2 (VBUS1), U29.C3 (A1), U29.D2 (VBUS2), U29.D3 (A0), U30.A2 (VBUS1), U30.D2 (VBUS2), C79.1, Q9.2 (E), R191.2
- net VDD_ISO_3: now also U30.C3 (A1), C80.1, Q11.2 (E), R192.2, U36.12
- net +12V_LDO_EN: now reaches U24.2 (EN)
- net +12V_LDO_EN: now also U27.11, R193.2
- net +15V_LDO_EN: now reaches U25.2 (EN)
- net +15V_LDO_EN: now also R194.2, U36.11
- net Current shunt/INPUT_CURRENT: now reaches C75.1, U23.10 (VOUT), U23.8 (VOUT), U23.9 (VOUT)
- net +5V_LDO_EN: now reaches U23.2 (EN)
- net +5V_LDO_EN: now also U26.11, R189.2
- net +INA_ISO_+5V: now reaches U28.A1 (IN+1)
- net -INA_ISO_+5V: now reaches U28.B1 (IN-1)
- net -INA_ISO_-5V: now reaches U28.C1 (IN-2)
- net +INA_ISO_-5V: now reaches U28.D1 (IN+2)
- net +INA_ISO_+12V: now reaches U29.A1 (IN+1)
- net -INA_ISO_+12V: now reaches U29.B1 (IN-1)
- net -INA_ISO_-12V: now reaches U29.C1 (IN-2)
- net +INA_ISO_-12V: now reaches U29.D1 (IN+2)
- net at U27.1: now also R195.2
- net -12V_LDO_EN: now reaches U27.10
- net -12V_LDO_EN: now also R161.1, R191.1
- net -12V_SCALE_IO_EXP: now reaches U27.13
- net -12V_SCALE_IO_EXP: now also U43.13 (P10_B)
- net at U27.14: now also R210.1
- net +12V_SCALE_IO_EXP: now reaches U27.15
- net +12V_SCALE_IO_EXP: now also U43.11 (P07_B)
- net at U27.16: now also R209.1
- net at U27.3: now also R196.2
- net at U27.5: now also R206.2
- net at U27.7: now also R208.2
- net +INA_ISO_+15V: now reaches U30.A1 (IN+1)
- net -INA_ISO_+15V: now reaches U30.B1 (IN-1)
- net -INA_ISO_-15V: now reaches U30.C1 (IN-2)
- net +INA_ISO_-15V: now reaches U30.D1 (IN+2)
- net at U26.1: now also R187.2
- net -5V_LDO_EN: now reaches U26.10
- net -5V_LDO_EN: now also R167.1, R190.1
- net -5V_SCALE_IO_EXP: now reaches U26.13
- net -5V_SCALE_IO_EXP: now also U43.8 (P04_B)
- net at U26.14: now also R204.1
- net +5V_SCALE_IO_EXP: now reaches U26.15
- net +5V_SCALE_IO_EXP: now also U43.7 (P03_B)
- net at U26.16: now also R203.1
- net at U26.3: now also R188.2
- net at U26.5: now also R205.2
- net at U26.7: now also R207.2
- net 12V_EN renamed 12V_ISO_EN
- net 12V_ISO_EN: now also U43.5 (P01_B)
- net 15V_EN renamed 15V_ISO_EN
- net 15V_ISO_EN: now also U43.6 (P02_B)
- net 5V_EN renamed 5V_ISO_EN
- net 5V_ISO_EN: now also U43.4 (P00_B)
- new net: C211.1, Q9.1 (B), R161.2
- new net: C213.1, Q23.1 (B), R167.2
- new net: Q11.3 (C), R165.1
- new net: Q12.3 (G), R165.2, R166.1
- new net: Q10.3 (G), R162.1, R163.2
- new net: R211.2, U36.5
- new net: R201.2, U36.1
- new net: Q9.3 (C), R163.1
- new net: C212.1, Q11.1 (B), R164.2
- new net: Q23.3 (C), R168.1
- new net: Q14.4 (G), R168.2, R169.1
- new net: R202.2, U36.3
- new net: R214.1, U36.14
- new net: R213.1, U36.16
- new net: R212.2, U36.7
- new net +12V_LDO_EN_IO_EXP: R206.1, U43.14 (P11_B)
- new net +15V_LDO_EN_IO_EXP: R211.1, U43.18 (P15_B)
- new net +15V_SCALE_IO_EXP: U36.15, U43.16 (P13_B)
- new net +5V_LDO_EN_IO_EXP: R205.1, U43.9 (P05_B)
- new net -12V_LDO_EN_IO_EXP: R208.1, U43.15 (P12_B)
- new net -15V_LDO_EN: R164.1, R192.1, U36.10
- new net -15V_LDO_EN_IO_EXP: R212.1, U43.19 (P16_B)
- new net -15V_SCALE_IO_EXP: U36.13, U43.17 (P14_B)
- new net -5V_LDO_EN_IO_EXP: R207.1, U43.10 (P06_B)
- new net Current shunt6/INPUT_CURRENT: C115.1, Q10.1 (D), Q10.2 (D), Q10.5 (D), Q10.6 (D), R177.2
- new net Current shunt7/INPUT_CURRENT: C112.1, Q12.1 (D), Q12.2 (D), Q12.5 (D), Q12.6 (D), R178.2
- new net ISO_+12V_SCALE: R195.1
- new net ISO_+15V_SCALE: R201.1
- new net ISO_+5V_SCALE: R187.1
- new net ISO_-12V_SCALE: R196.1
- new net ISO_-15V_SCALE: R202.1
- new net ISO_-5V_SCALE: R188.1
- new net Isolated dual rail PS controlled submodule/+ISO_LDO_CTRL_x1_+15V_SCALE: U67.4 (P00_B)
- new net Isolated dual rail PS controlled submodule/+ISO_LDO_CTRL_x2_+15V_SCALE: U67.5 (P01_B)
- new net Isolated dual rail PS controlled submodule/+PWR_SWITCH_ISO_CTRL_X1_EN: U67.8 (P04_B)
- new net Isolated dual rail PS controlled submodule/+PWR_SWITCH_ISO_CTRL_X2_EN: U67.9 (P05_B)
- new net Isolated dual rail PS controlled submodule/-ISO_LDO_CTRL_x1_+15V_SCALE: U67.6 (P02_B)
- new net Isolated dual rail PS controlled submodule/-ISO_LDO_CTRL_x2_+15V_SCALE: U67.7 (P03_B)
- new net Isolated dual rail PS controlled submodule/-PWR_SWITCH_ISO_CTRL_1X_EN: U67.10 (P06_B)
- new net Isolated dual rail PS controlled submodule/-PWR_SWITCH_ISO_CTRL_2X_EN: U67.11 (P07_B)
- new net Isolated dual rail PS controlled submodule1/+ISO_LDO_CTRL_x1_+15V_SCALE: U67.13 (P10_B)
- new net Isolated dual rail PS controlled submodule1/+ISO_LDO_CTRL_x2_+15V_SCALE: U67.14 (P11_B)
- new net Isolated dual rail PS controlled submodule1/+PWR_SWITCH_ISO_CTRL_X1_EN: U67.17 (P14_B)
- new net Isolated dual rail PS controlled submodule1/+PWR_SWITCH_ISO_CTRL_X2_EN: U67.18 (P15_B)
- new net Isolated dual rail PS controlled submodule1/-ISO_LDO_CTRL_x1_+15V_SCALE: U67.15 (P12_B)
- new net Isolated dual rail PS controlled submodule1/-ISO_LDO_CTRL_x2_+15V_SCALE: U67.16 (P13_B)
- new net Isolated dual rail PS controlled submodule1/-PWR_SWITCH_ISO_CTRL_1X_EN: U67.19 (P16_B)
- new net Isolated dual rail PS controlled submodule1/-PWR_SWITCH_ISO_CTRL_2X_EN: U67.20 (P17_B)
- no-connect marks 15 -> 17
Other:
- removed sheet Current shunt2
- removed sheet Current shunt3
- added sheet Current shunt6 (current_sensing.kicad_sch)
- added sheet Current shunt7 (current_sensing.kicad_sch)
- sheet Isolated dual rail PS controlled submodule ports: added +ISO_LDO_CTRL_x1_+15V, +ISO_LDO_CTRL_x1_+15V_SCALE, +ISO_LDO_CTRL_x2_+15V, +ISO_LDO_CTRL_x2_+15V_SCALE, +PWR_SWITCH_ISO_CTRL_X1_EN, +PWR_SWITCH_ISO_CTRL_X2_EN, -ISO_LDO_CTRL_x1_+15V, -ISO_LDO_CTRL_x1_+15V_SCALE, -ISO_LDO_CTRL_x2_+15V, -ISO_LDO_CTRL_x2_+15V_SCALE, -PWR_SWITCH_ISO_CTRL_1X_EN, -PWR_SWITCH_ISO_CTRL_2X_EN, INA_A0, INA_A1, SCL_ISO, SDA_ISO; removed none
- sheet Isolated dual rail PS controlled submodule1 ports: added +ISO_LDO_CTRL_x1_+15V, +ISO_LDO_CTRL_x1_+15V_SCALE, +ISO_LDO_CTRL_x2_+15V, +ISO_LDO_CTRL_x2_+15V_SCALE, +PWR_SWITCH_ISO_CTRL_X1_EN, +PWR_SWITCH_ISO_CTRL_X2_EN, -ISO_LDO_CTRL_x1_+15V, -ISO_LDO_CTRL_x1_+15V_SCALE, -ISO_LDO_CTRL_x2_+15V, -ISO_LDO_CTRL_x2_+15V_SCALE, -PWR_SWITCH_ISO_CTRL_1X_EN, -PWR_SWITCH_ISO_CTRL_2X_EN, INA_A0, INA_A1, SCL_ISO, SDA_ISO; removed none
- note added: "I2C ID: 0x44"
- note added: "I2C ID: 0x45"
- note added: "I2C ID: 0x46"
- note added: "I2C ID: 0x47"
- note added: "I2C ID: 0x48"
- note added: "Notes to the future self: - Negative enable mus be labeled as negated eg:. ~{-5V_LDO_EN} - Check for current consumption for the negated EN. Since the 50mA Opto forward current seems a lot - Check for current consumption for the Negative Power Switch, since it pulls 50mA as well - Still needs to place I2C IDs"
- note removed: "Needs to set the I2C ID"
- moved on the sheet: C39, C40, C41, C42, C43, C44, C45, C46, C47, C48, C49, C50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

Commit message: HW-61/chore: Added simulation for switch ocntrol, organized the overall schematic, fixed the ERC errors. Still pending for the current sense components and negative side LDO control
Parts:
- removed C211, C212, C213: 1uF-0402_01, passive:Capacitor_0402, symbol capacitor:1uF-0402_01
- added C211, C212, C213: 100nF-0402_01, passive:Capacitor_0402, symbol capacitor:100nF-0402_01
Connections:
- net +5V: now also U43.2 (A1); no longer U67.24 (VDD)
- net 15V_SCL_ISO: now also U67.22 (SCL)
- net 15V_SDA_ISO: now also U67.23 (SDA)
- net GND: now also U43.21 (A0), U43.3 (A2); no longer U67.12 (GND)
- net GND_ISO_12V: now also C211.2
- net GND_ISO_15V: now also U67.12 (GND), U67.3 (A2), C212.2
- net GND_ISO_5V: now also C213.2
- net VDD_ISO_1: no longer U20.12 (VISO)
- net VDD_ISO_2: no longer U21.12 (VISO)
- net VDD_ISO_3: now also U67.2 (A1), U67.21 (A0), U67.24 (VDD); no longer U22.12 (VISO)
- net at Q9.1 (B), R161.2: now also C211.1
- net at Q23.1 (B), R167.2: now also C213.1
- net at Q11.1 (B), R164.2: now also C212.1
- net -12V_LDO_EN renamed ~{-12V_LDO_EN}
- net -15V_LDO_EN renamed ~{-15V_LDO_EN}
- net -5V_LDO_EN renamed ~{-5V_LDO_EN}
- net Isolated dual rail PS controlled submodule/-PWR_SWITCH_ISO_CTRL_1X_EN renamed Isolated dual rail PS controlled submodule/~{-PWR_SWITCH_ISO_CTRL_1X_EN}
- net Isolated dual rail PS controlled submodule/-PWR_SWITCH_ISO_CTRL_2X_EN renamed Isolated dual rail PS controlled submodule/~{-PWR_SWITCH_ISO_CTRL_2X_EN}
- net Isolated dual rail PS controlled submodule1/-PWR_SWITCH_ISO_CTRL_1X_EN renamed Isolated dual rail PS controlled submodule1/~{-PWR_SWITCH_ISO_CTRL_1X_EN}
- net Isolated dual rail PS controlled submodule1/-PWR_SWITCH_ISO_CTRL_2X_EN renamed Isolated dual rail PS controlled submodule1/~{-PWR_SWITCH_ISO_CTRL_2X_EN}
- net SCL renamed SCL_B
- net SCL_B: no longer U43.22 (SCL), U67.22 (SCL)
- net SDA renamed SDA_B
- net SDA_B: no longer U43.23 (SDA), U67.23 (SDA)
- new net SCL_A: U43.22 (SCL)
- new net SDA_A: U43.23 (SDA)
- no-connect marks 17 -> 18
Other:
- sheet Isolated dual rail PS controlled submodule ports: added DigiPot_A0, DigiPot_A1, DigiPot_A2, ~{-PWR_SWITCH_ISO_CTRL_1X_EN}, ~{-PWR_SWITCH_ISO_CTRL_2X_EN}; removed -PWR_SWITCH_ISO_CTRL_1X_EN, -PWR_SWITCH_ISO_CTRL_2X_EN
- sheet Isolated dual rail PS controlled submodule1 ports: added DigiPot_A0, DigiPot_A1, DigiPot_A2, ~{-PWR_SWITCH_ISO_CTRL_1X_EN}, ~{-PWR_SWITCH_ISO_CTRL_2X_EN}; removed -PWR_SWITCH_ISO_CTRL_1X_EN, -PWR_SWITCH_ISO_CTRL_2X_EN
- note added: "I2C ID: 0x22"
- note added: "I2C ID: 0x23"
- note added: "INA I2C ID: 0x47 DigiPot ID: 0x52"
- note added: "INA I2C ID: 0x48 DigiPot ID: 0x53"
- note added: "Notes to the future self: - Check for current consumption for the negated EN. Since the 50mA Opto forward current seems a lot - Check for current consumption for the Negative Power Switch, since it pulls 50mA as well - Replace 1u to 100n"
- note removed: "I2C ID: 0x47"
- note removed: "I2C ID: 0x48"
- note removed: "Notes to the future self: - Negative enable mus be labeled as negated eg:. ~{-5V_LDO_EN} - Check for current consumption for the negated EN. Since the 50mA Opto forward current seems a lot - Check for current consumption for the Negative Power Switch, since it pulls 50mA as well - Still needs to place I2C IDs"
- moved on the sheet: C112, C115, C39, C40, C45, C48, C51, C76, R167, R190, R191, R192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
