File: powerboard.kicad_sch (KiCad schematic)
At the start: 2 parts, among them J1 1-1939638-7, J2 1-1939638-7

Commit message: HW-61 chore: FT4233 Wire'd up
Parts:
- added C176, C179, C180, C183, C184, C185, C186, C187, C188, C189, C190, C191, C192, C195: 100nF-0402_01, passive:Capacitor_0402, symbol capacitor:100nF-0402_01
- added C177, C178: 16pF-0402_01, passive:Capacitor_0402, symbol capacitor:16pF-0402_01
- added C181, C182, C193, C194: 1uF-0402_01, passive:Capacitor_0402, symbol capacitor:1uF-0402_01
- added D5, D6, D7: BAT760-7, semiconductor:SOD323-2_P2.2_1.7x1.25x0.95, symbol semiconductor:BAT760-7
- added JP2: SolderJumper_2_Bridged, electromechanical:SolderJumper_2_NBridged, symbol electromechanical:SolderJumper_2_NBridged
- added R142: 10k-0402_02, passive:Resistor_0402, symbol resistor:10k-0402_02
- added R143: 2k-0402_01, passive:Resistor_0402, symbol resistor:2k-0402_01
- added R144, R145, R146: 10k-0402_01, passive:Resistor_0402, symbol resistor:10k-0402_01
- added R147: 12k-0402_01, passive:Resistor_0402, symbol resistor:12k-0402_01
- added R148, R151, R152, R153, R154: 1k-0402_01, passive:Resistor_0402, symbol resistor:1k-0402_01
- added R149: 100k-0402_01, passive:Resistor_0402, symbol resistor:100k-0402_01
- added R150: 15.8k-0402_01, passive:Resistor_0402, symbol resistor:15.8k-0402_01
- added U1: FT4233HP, semiconductor:QFN-76-1EP_P0.4_9x9x0.9, symbol integrated-circuit:FT4233HP
- added U2: USB2512BT/M2, semiconductor:SQFN-36-1EP_P0.5_6x6x0.9, symbol integrated-circuit:USB2512BT/M2
- added U3: M24C02-FMC6TG, semiconductor:UFDFPN-8-1EP_P0.5_2x3x0.55, symbol integrated-circuit:M24C02-FMC6TG
- added U65: 93LC56BT-I/OT, semiconductor:SOT23-6_P0.95_2.925x1.625x1.175, symbol integrated-circuit:93LC56BT-I/OT
- added U66: AP2127K-3.3TRG1, semiconductor:SOT23-5_P0.95_2.9x1.6x1.18, symbol integrated-circuit:AP2127K-3.3TRG1
- added Y1: ECS-120-8-36-CKM, passive:ECX-2236, symbol oscilator:ECS-120-8-36-CKM
Connections:
- new net: R148.2, U1.4 (RESET#)
- new net: C178.1, U1.30 (OSCO), Y1.3
- new net: R145.1, U1.1 (EECLK), U65.4 (CLK)
- new net: R143.2, U1.2 (EEDATA), U65.3 (DI)
- new net: C177.1, U1.29 (OSCI), Y1.1
- new net: R147.2, U1.65 (REF)
- new net: R144.1, U1.76 (EECS), U65.5 (CS)
- new net: R143.1, R146.1, U65.1 (DO)
- new net: D7.1 (Cathode), U1.20 (BDBUS1-RXD)
- new net: JP2.2 (B), R142.2, U3.7 (~{WC})
- new net: R149.1, R150.2, U1.68 (PD1_SVBUS)
- new net: D6.1 (Cathode), U1.9 (ADBUS1-RXD)
- new net +1V2: C188.1, C189.1, C190.1, C191.1, C192.1, U1.10 (VCORE), U1.27 (VCORE), U1.33 (VREGOUT), U1.47 (VCORE), U1.74 (VCORE)
- new net +3V3: C179.1, C180.1, C182.1, C194.1, D5.2 (Anode), R144.2, R145.2, R146.2, R148.1, R151.2, R152.2, R153.2, R154.2, U1.66 (VCC_PD), U65.6 (VCC), U66.5 (VOUT)
- new net +3V3_FTDI: C183.1, C184.1, C185.1, C186.1, C187.1, C193.1, C195.1, D5.1 (Cathode), U1.12 (VCCIO), U1.28 (VCCIO), U1.32 (VREGIN), U1.41 (VCCIO), U1.54 (VCCIO), U1.62 (VCC_USB), U1.69 (PD1_VCONN)
- new net +5V: C176.1, C181.1, R142.1, R149.2, U3.8 (VCC), U66.1 (VIN), U66.3 (~{SHUTDOWN})
- new net GND: C176.2, C177.2, C178.2, C179.2, C180.2, C181.2, C182.2, C183.2, C184.2, C185.2, C186.2, C187.2, C188.2, C189.2, C190.2, C191.2, C192.2, C193.2, C194.2, C195.2, JP2.1 (A), R147.1, R150.1, U1.11 (GND), U1.3 (TEST), U1.31 (GND), U1.55 (GND), U1.77 (EP), U3.4 (VSS), U3.9 (EPAD), U65.2 (VSS), U66.2 (GND), Y1.2, Y1.4
- new net SCL: U3.6 (SCL)
- new net SCL_PRE_LVL_SHIFTER_B: R152.1, R154.1, U1.19 (BDBUS0-TXD), U1.8 (ADBUS0-TXD)
- new net SDA: U3.5 (SDA)
- new net SDA_PRE_LVL_SHIFTER_B: D6.2 (Anode), D7.2 (Anode), R151.1, R153.1, U1.13 (ADBUS2-RTS#), U1.21 (BDBUS2-RTS#)
- new net USB_HUB_N: U1.63 (DM)
- new net USB_HUB_P: U1.64 (DP)
- no-connect marks 0 -> 43
Other:
- sheet Isolated dual rail fixed PS stage renamed Isolated dual rail PS stage
- removed sheet Isolated dual rail controlled PS stage
- note added: ""DO/DI - Wired together and connected to SDA pin of 24LC256 for bidirectional data transfer. DO set as output pin to transfer serial data or address from FT2232H to 24LC256 device. DI set as input pin to receive serial data input pin from 24LC256 device to FT2232H. Requires a pull-up resistor to VCC (typical 10 KΩ for 100 kHz and 2 KΩ for 400 kHz). ""
- note added: "Schottky diode so the DO can only pull the SDA low. Replace for 0R if this goes south"
- note added: "Start with 1k to try run the Bus at 1Mhz."

Commit message: HW-61 chore: Added a simple comment
Other:
- note added: "Test using the FT4233 GPIOs to control and read states of the INA scales. But use it as a redundant feature, still maintain the IO/Expanders as main drivers"
Changed lines of the file:
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@@
+		)
+	)
+	(text "Test using the FT4233 GPIOs to control and read states of the INA scales.\nBut use it as a redundant feature, still maintain the IO/Expanders as main\ndrivers"
+		(exclude_from_sim no)
+		(at 66.802 372.618 0)
+		(effects
+			(font
+				(size 0.762 0.762)
+			)
+			(justify left)
 		)
 	)

Commit message: Details to finish
Parts:
- added C196, C197, C198, C199, C200, C201, C204, C206, C207: 100nF-0402_01, passive:Capacitor_0402, symbol capacitor:100nF-0402_01
- added C202: 4.7uF-1206_02, passive:Capacitor_1206, symbol capacitor:4.7uF-1206_02
- added C203, C205, C208: 1uF-0402_01, passive:Capacitor_0402, symbol capacitor:1uF-0402_01
- added C209, C210: 18pF-0402_01, passive:Capacitor_0402, symbol capacitor:18pF-0402_01
- added D10, D11, D12, D14, D15, D16, D17, D18, D19, D20, D22, D23, D24, D25, D26, D27, D28, D29, D30, D31, D32, D33, D34, D38, D8, D9: SMAJ20A, staging:DO-214AC_P3.97_4.24x2.67x2.25mm, symbol staging:SMAJ20A
- added D13, D36, D37: D30V0S1UG3LP20-7, semiconductor:UDFN2020-3_P0.65_2x2x0.6, symbol semiconductor:D30V0S1UG3LP20-7
- added D21: ESD122DMYR, semiconductor:X2SON-3_P0.5_1.32x0.6x0.4, symbol semiconductor:ESD122DMYR
- added D35, D39, D69: SMBJ7.0A-13-F, semiconductor:SMB-2_P4.3_4.315x3.62x2.25, symbol semiconductor:SMBJ7.0A-13-F
- added D40, D41: SMAJ60A, staging:DO-214AC_P3.97_4.24x2.67x2.25mm, symbol staging:SMAJ60A
- added J3: HSEC8-120-01-S-DV-A-K-TR_PCIe, custom:HSEC8-120-01-S-DV-A-K-TR_PCIe, symbol custom:HSEC8-120-01-S-DV-A-K-TR_PCIe
- added R155: 12k-0402_01, passive:Resistor_0402, symbol resistor:12k-0402_01
- added R156, R157, R158, R159: 100k-0402_01, passive:Resistor_0402, symbol resistor:100k-0402_01
- added R160: 1M-0402_01, passive:Resistor_0402, symbol resistor:1M-0402_01
- added Y2: TSX-3225_24.0000MF20G-AC3, passive:TSX-3225, symbol oscilator:TSX-3225_24.0000MF20G-AC3
Connections:
- net USB_HUB_N is gone; now on net FT_USB_HUB_N: U1.63 (DM)
- net USB_HUB_P is gone; now on net FT_USB_HUB_P: U1.64 (DP)
- net +3V3: now also U2.10 (VDDA33), U2.15 (VDD33), U2.23 (VDD33), U2.29 (VDDA33), U2.36 (VDDA33), U2.5 (VDDA33), C196.1, C197.1, C198.1, C199.1, C200.1, C201.1, C202.1, R156.2
- net +5V: now also J2.A15, C208.1, D69.1 (Cathode), J3.11, J3.7, J3.9, R158.1
- net GND: now also J1.1, J1.2, J1.B10, J1.B11, J1.B12, J1.B13, J1.B14, J1.B15, J1.B16, J1.B17, J1.B2, J1.B3, J1.B4, J1.B5, J1.B6, J1.B7, J1.B8, J1.B9, J2.1, J2.2, J2.B16, J2.B17, U2.37 (VSS), C196.2, C197.2, C198.2, C199.2, C200.2, C201.2, C202.2, C203.2, C204.2, C205.2, C206.2, C207.2, C208.2, C209.2, C210.2, D10.2, D11.2, D12.2, D13.3 (Anode), D14.2, D15.2, D16.2, D17.2, D18.2, D19.2, D20.2, D21.1 (GND), D21.1 (GND), D22.2, D23.2, D24.2, D26.2, D40.2 (Anode), D41.1 (Cathode), D69.2 (Anode), D8.2, D9.2, J3.10, J3.12, J3.18, J3.2, J3.20, J3.22, J3.24, J3.26, J3.28, J3.30, J3.32, J3.34, J3.36, J3.38, J3.4, J3.40, J3.6, J3.8, R155.1, R157.1, R159.2, Y2.2, Y2.4
- net SCL: now also J3.16
- net SDA: now also J3.14
- net FT_USB_HUB_N: now reaches U2.1 (USBDM_DN1)
- net FT_USB_HUB_P: now reaches U2.2 (USBDP_DN1)
- net at U2.27 (VBUS_DET): now also R158.2, R159.1
- net OUT_USB_HUB_N: now reaches U2.3 (USBDM_DN2)
- net OUT_USB_HUB_N: now also J1.A1
- net UPSTREAM_N: now reaches U2.30 (USBDM_UP)
- net UPSTREAM_N: now also D21.3 (IO2), J3.31
- net UPSTREAM_P: now reaches U2.31 (USBDP_UP)
- net UPSTREAM_P: now also D21.2 (IO1), J3.29
- net OUT_USB_HUB_P: now reaches U2.4 (USBDP_DN2)
- net OUT_USB_HUB_P: now also J1.B1
- net GND_ISO_15V: now reaches J2.A1
- net GND_ISO_15V: now also J2.A11, J2.A13, J2.A7, J2.A9, J2.B1, J2.B11, J2.B13, J2.B7, J2.B9, D25.2, D27.2, D28.2, D29.2, D30.2, D31.1, D32.1, D33.1, D34.1, D38.1
- net +ISO_LDO_CTRL_x2_+15V_CH21: now reaches J2.A10
- net +ISO_LDO_CTRL_x2_+15V_CH21: now also D28.1
- net +ISO_LDO_CTRL_x1_+15V_CH22: now reaches J2.A12
- net +ISO_LDO_CTRL_x1_+15V_CH22: now also D30.1
- net +ISO_LDO_CTRL_x2_+15V_CH23: now reaches J2.A14
- net +ISO_LDO_CTRL_x2_+15V_CH23: now also D29.1
- net BOOST_50V_CH25: now reaches J2.A16
- net BOOST_50V_CH25: now also D40.1 (Cathode)
- net BOOST_50V_CH26: now reaches J2.A17
- net BOOST_50V_CH26: now also D41.2 (Anode)
- net ISO_+15V_CH17: now reaches J2.A2
- net ISO_+15V_CH17: now also D25.1
- net GND_ISO_12V: now reaches J2.A3
- net GND_ISO_12V: now also J2.B3, D36.3 (Anode), D37.1 (Cathode), D37.2 (Cathode)
- net ISO_+12V_CH18: now reaches J2.A4
- net ISO_+12V_CH18: now also D36.1 (Cathode), D36.2 (Cathode)
- net GND_ISO_5V: now reaches J2.A5
- net GND_ISO_5V: now also J2.B5, D35.2 (Anode), D39.1 (Cathode)
- net ISO_+5V_CH19: now reaches J2.A6
- net ISO_+5V_CH19: now also D35.1 (Cathode)
- net +ISO_LDO_CTRL_x1_+15V_CH20: now reaches J2.A8
- net +ISO_LDO_CTRL_x1_+15V_CH20: now also D27.1
- net -ISO_LDO_CTRL_x2_+15V_CH21: now reaches J2.B10
- net -ISO_LDO_CTRL_x2_+15V_CH21: now also D32.2
- net -ISO_LDO_CTRL_x1_+15V_CH22: now reaches J2.B12
- net -ISO_LDO_CTRL_x1_+15V_CH22: now also D33.2
- net -ISO_LDO_CTRL_x2_+15V_CH23: now reaches J2.B14
- net -ISO_LDO_CTRL_x2_+15V_CH23: now also D34.2
- net +24V: now reaches J2.B15
- net +24V: now also D13.1 (Cathode), D13.2 (Cathode), J3.1, J3.3, J3.5
- net ISO_-15V_CH17: now reaches J2.B2
- net ISO_-15V_CH17: now also D38.2
- net ISO_-12V_CH18: now reaches J2.B4
- net ISO_-12V_CH18: now also D37.3 (Anode)
- net ISO_-5V_CH19: now reaches J2.B6
- net ISO_-5V_CH19: now also D39.2 (Anode)
- net -ISO_LDO_CTRL_x1_+15V_CH20: now reaches J2.B8
- net -ISO_LDO_CTRL_x1_+15V_CH20: now also D31.2
- net at U2.14 (CRFILT): now also C205.1, C206.1
- net at U2.32 (XTALOUT): now also C209.1, R160.2, Y2.1
- net at U2.33 (XTALIN): now also C210.1, R160.1, Y2.3
- net at U2.34 (PLLFILT): now also C203.1, C204.1
- net at U2.35 (RBIAS): now also R155.2
- net at U2.26 (RESET_N): now also C207.1, R156.1
- net at U2.28 (SUSP_IND): now also R157.2
- net BUCK_CH9: now reaches J1.A10
- net BUCK_CH9: now also D17.1
- net BUCK_CH10: now reaches J1.A11
- net BUCK_CH10: now also D18.1
- net BUCK_CH11: now reaches J1.A12
- net BUCK_CH11: now also D19.1
- net BUCK_CH12: now reaches J1.A13
- net BUCK_CH12: now also D20.1
- net BUCK_CH13: now reaches J1.A14
- net BUCK_CH13: now also D22.1
- net BUCK_CH14: now reaches J1.A15
- net BUCK_CH14: now also D23.1
- net BUCK_CH15: now reaches J1.A16
- net BUCK_CH15: now also D24.1
- net BUCK_CH16: now reaches J1.A17
- net BUCK_CH16: now also D26.1
- net BUCK_CH1: now reaches J1.A2
- net BUCK_CH1: now also D8.1
- net BUCK_CH2: now reaches J1.A3
- net BUCK_CH2: now also D9.1
- net BUCK_CH3: now reaches J1.A4
- net BUCK_CH3: now also D10.1
- net BUCK_CH4: now reaches J1.A5
- net BUCK_CH4: now also D11.1
- net BUCK_CH5: now reaches J1.A6
- net BUCK_CH5: now also D12.1
- net BUCK_CH6: now reaches J1.A7
- net BUCK_CH6: now also D14.1
- net BUCK_CH7: now reaches J1.A8
- net BUCK_CH7: now also D15.1
- net BUCK_CH8: now reaches J1.A9
- net BUCK_CH8: now also D16.1
- no-connect marks 43 -> 62
Other:
- note added: ""DO/DI - Wired together and connected to SDA pin of ]24LC256 for bidirectional data transfer. DO set as output pin to transfer serial data or address from FT2232H to 24LC256 device. DI set as input pin to receive serial data input pin from 24LC256 device to FT2232H. Requires a pull-up resistor to VCC (typical 10 KΩ for 100 kHz and 2 KΩ for 400 kHz). ""
- note added: "Calculate the trace capacitance and replace the 18pF for a more appropriate value"
- note added: "Cb1 = Trace capacitance 1 Cxtal = 6pF Cs1 = Cb1 + Cxtal Cb2 = Trace capacitance 2 Cxtal = 6pF Cs2 = Cb2 + Cxtal Cl = 18pF C0 = 3pF"
- note removed: ""DO/DI - Wired together and connected to SDA pin of 24LC256 for bidirectional data transfer. DO set as output pin to transfer serial data or address from FT2232H to 24LC256 device. DI set as input pin to receive serial data input pin from 24LC256 device to FT2232H. Requires a pull-up resistor to VCC (typical 10 KΩ for 100 kHz and 2 KΩ for 400 kHz). ""
- moved on the sheet: C176, C177, C178, C179, C180, C181, C182, C183, C184, C185, C186, C187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

Commit message: HW-61/chore: Added simulation for switch ocntrol, organized the overall schematic, fixed the ERC errors. Still pending for the current sense components and negative side LDO control
Parts:
- added R234, R235, R239, R240: 1k-0402_01, passive:Resistor_0402, symbol resistor:1k-0402_01
- added R237, R238: 200k-0402_01, passive:Resistor_0402, symbol resistor:200k-0402_01
- added U69, U70: PCA9306DQER, staging:DQE8_P0.35_1.00x1.415x0.37mm, symbol staging:PCA9306DQER
- D13: Criticality (none) -> C/S/G; Lead Time (W) (none) -> LT; Maturity Level (none) -> P/V/F; PLM Code TBD -> PRPTRAC00000777
- D21: Criticality (none) -> C/S/G; Lead Time (W) (none) -> LT; Maturity Level (none) -> P/V/F; PLM Code TBD -> PRPTRAC00000780
- D35, D39, D69: Criticality (none) -> C/S/G; Lead Time (W) (none) -> LT; Maturity Level (none) -> P/V/F; SAP Code TBD -> DIOT-XXXX
- J3: Criticality (none) -> C/S/G; Lead Time (W) (none) -> LT; Maturity Level (none) -> P/V/F
- JP2: Criticality (none) -> NA; Lead Time (W) (none) -> NA; Maturity Level (none) -> NA
Connections:
- net +3V3: now also U69.2 (Vref1), U70.2 (Vref1)
- net +5V: now also R234.2, R235.2, R237.2, R238.2, R239.2, R240.2
- net GND: now also U3.1 (E0), U3.2 (E1), U3.3 (E2), U69.1 (GND), U70.1 (GND)
- net SCL_PRE_LVL_SHIFTER_B: now also U70.3 (SCL1); no longer R154.1, U1.8 (ADBUS0-TXD)
- net SDA_PRE_LVL_SHIFTER_B: now also U70.4 (SDA1); no longer D6.2 (Anode), R153.1, U1.13 (ADBUS2-RTS#)
- new net: R237.1, U69.7 (Vref2), U69.8 (EN)
- new net: R238.1, U70.7 (Vref2), U70.8 (EN)
- new net SCL_A: R235.1, U69.6 (SCL2)
- new net SCL_B: R240.1, U70.6 (SCL2)
- new net SCL_PRE_LVL_SHIFTER_A: R154.1, U1.8 (ADBUS0-TXD), U69.3 (SCL1)
- new net SDA_A: R234.1, U69.5 (SDA2)
- new net SDA_B: R239.1, U70.5 (SDA2)
- new net SDA_PRE_LVL_SHIFTER_A: D6.2 (Anode), R153.1, U1.13 (ADBUS2-RTS#), U69.4 (SDA1)
Other:
- note added: "1kOhm resistors for 1 Mbps application"
- moved on the sheet: C207, R156, R157, U2B
